Commit message: Modify PD gains and urdf file

File: source/isaac_lab_actuator_dynamic/isaac_lab_actuator_dynamic/assets/urdf/leg05/hr.urdf (robot description, URDF)
Before this commit: robot hr, 13 links, 12 joints
Joints:
- joint L_calf_joint: limit lower=0 upper=2.1 effort=300 velocity=50 -> lower=-1.571 upper=0.529 effort=300 velocity=50; origin xyz=0 0 -0.35 rpy=0 0 0 -> xyz=0 0 -0.35 rpy=0 1.571 0
- joint L_thigh_joint: limit lower=-2.05 upper=0 effort=300 velocity=50 -> lower=-1.26 upper=0.78 effort=300 velocity=50; origin xyz=0.078 -0.014084 -0.0185 rpy=0 0 0 -> xyz=0.078 -0.014084 -0.0185 rpy=0 -0.78539816339 0
- joint L_toe_joint: origin xyz=0 0 -0.35 rpy=0 0 0 -> xyz=0 0 -0.35 rpy=0 -0.78539815339 0
- joint R_calf_joint: limit lower=0 upper=2.1 effort=300 velocity=50 -> lower=-1.571 upper=0.529 effort=300 velocity=50; origin xyz=0 0 -0.35 rpy=0 0 0 -> xyz=0 0 -0.35 rpy=0 1.571 0
- joint R_thigh_joint: limit lower=-2.05 upper=0 effort=300 velocity=50 -> lower=-1.76 upper=0.78 effort=300 velocity=50; origin xyz=0.078 0.014084 -0.0185 rpy=0 0 0 -> xyz=0.078 0.014084 -0.0185 rpy=0 -0.78539816339 0
- joint R_toe_joint: origin xyz=0 0 -0.35 rpy=0 0 0 -> xyz=0 0 -0.35 rpy=0 -0.78539815339 0

Commit message: fine tune reward scales

File: source/isaac_lab_actuator_dynamic/isaac_lab_actuator_dynamic/assets/urdf/leg05/hr.urdf (robot description, URDF)
Before this commit: robot hr, 13 links, 12 joints
Links:
- link L_calf: geometry collision cylinder length=0.27 radius=0.04; visual mesh filename=meshes/L_calf.STL
- link L_thigh: geometry collision cylinder length=0.30 radius=0.04; visual mesh filename=meshes/L_thigh.STL
- link R_calf: geometry collision cylinder length=0.30 radius=0.04; visual mesh filename=meshes/R_calf.STL
- link R_thigh: geometry collision cylinder length=0.30 radius=0.04; visual mesh filename=meshes/R_thigh.STL
Joints:
- joint L_thigh_joint: limit lower=-1.26 upper=0.78 effort=300 velocity=50 -> lower=-1.26 upper=0.8 effort=300 velocity=50

Commit message: Fine tune the gait command

File: source/isaac_lab_actuator_dynamic/isaac_lab_actuator_dynamic/assets/urdf/leg05/hr.urdf (robot description, URDF)
Before this commit: robot hr, 13 links, 12 joints
Joints:
- joint L_calf_joint: limit lower=-1.571 upper=0.529 effort=300 velocity=50 -> lower=-1.571 upper=0.529 effort=105 velocity=50
- joint L_hip2_joint: limit lower=-0.5 upper=0.65 effort=300 velocity=50 -> lower=-0.26 upper=0.65 effort=125 velocity=50
- joint L_hip_joint: limit lower=-1.5 upper=1.5 effort=300 velocity=50 -> lower=-1.5 upper=1.5 effort=125 velocity=50
- joint L_thigh_joint: limit lower=-1.26 upper=0.8 effort=300 velocity=50 -> lower=-1.25 upper=1.1 effort=125 velocity=50
- joint L_toe_joint: limit lower=-0.8 upper=0.8 effort=100 velocity=50 -> lower=-0.3 upper=1.6 effort=30 velocity=50
- joint R_calf_joint: limit lower=-1.571 upper=0.529 effort=300 velocity=50 -> lower=-1.571 upper=0.529 effort=105 velocity=50
- joint R_hip2_joint: limit lower=-0.65 upper=0.5 effort=300 velocity=50 -> lower=-0.65 upper=0.26 effort=125 velocity=50
- joint R_hip_joint: limit lower=-1.5 upper=1.5 effort=300 velocity=50 -> lower=-1.5 upper=1.5 effort=125 velocity=50
- joint R_thigh_joint: limit lower=-1.76 upper=0.78 effort=300 velocity=50 -> lower=-1.25 upper=1.1 effort=125 velocity=50
- joint R_toe_joint: limit lower=-0.8 upper=0.8 effort=100 velocity=50 -> lower=-0.3 upper=1.6 effort=30 velocity=50

Commit message: First commit

File: source/isaac_lab_actuator_dynamic/isaac_lab_actuator_dynamic/assets/urdf/leg05/hr.urdf (robot description, URDF)
Before this commit: robot hr, 13 links, 12 joints
Links:
- link L_calf: mass 1.5 -> 1.326656
- link L_hip2: mass 1.33325 -> 1.726000
- link L_thigh: mass 4.91 -> 4.750102
- link L_toe: mass 0.52014 -> 0.520
- link R_calf: mass 1.5 -> 1.326656
- link R_hip2: mass 1.33325 -> 1.726000
- link R_thigh: mass 4.91 -> 4.750102
- link R_toe: mass 0.52014 -> 0.520
- link base: mass 13 -> 7.4
