Commit message: Add actuator dynamic model config

File: source/isaac_lab_actuator_dynamic/isaac_lab_actuator_dynamic/assets/urdf/leg00/leg00.urdf (robot description, URDF)
Before this commit: robot leg00, 13 links, 12 joints
Links:
- link L_toe: geometry collision mesh filename=meshes/L_toe.STL; visual mesh filename=meshes/L_toe.STL scale=1.0 1.0 0.5

File: source/isaac_lab_actuator_dynamic/isaac_lab_actuator_dynamic/assets/urdf/leg05/hr_newfoot.urdf (robot description, URDF)
Before this commit: robot hr, 13 links, 12 joints
Links:
- link L_toe: mass 0.520 -> 0.177100; geometry collision mesh filename=meshes/L_toe_newfoot.STL scale=1.0 1.0 0.5714; visual mesh filename=meshes/L_toe_newfoot.STL scale=1.0 1.0 0.5714
- link R_toe: mass 0.520 -> 0.177100; geometry collision mesh filename=meshes/R_toe_newfoot.STL scale=1.0 1.0 0.5714; visual mesh filename=meshes/R_toe_newfoot.STL scale=1.0 1.0 0.5714
- link base: mass 13.923 -> 7.4
