Commit message: Add Isaac Sim training

File: source/isaac_lab_actuator_dynamic/isaac_lab_actuator_dynamic/assets/urdf/Leg_Changed_IMU/Wholebody_URDF_IMU_Changed.urdf (robot description, URDF)
Before this commit: robot hr, 13 links, 12 joints
Links:
- removed link L_end_effector
- removed link R_end_effector
- removed link base
- added link Pelvis, mass 6.661487; collision box size=0.21 0.38 0.33; visual mesh filename=meshes/Pelvis.STL
- added link Torso, mass 1.561; visual mesh filename=meshes/Torso.STL
- link L_calf: geometry collision cylinder length=0.25 radius=0.04; visual mesh filename=meshes/L_calf.STL
- link L_hip: mass 1.5262 -> 1.544
- link L_thigh: geometry collision cylinder length=0.25 radius=0.04; visual mesh filename=meshes/L_thigh.STL
- link L_toe: geometry collision mesh filename=meshes/L_toe_old.STL; visual mesh filename=meshes/L_toe_old.STL
- link R_calf: geometry collision cylinder length=0.25 radius=0.04; visual mesh filename=meshes/R_calf.STL
- link R_hip: mass 1.5262 -> 1.544
- link R_thigh: geometry collision cylinder length=0.25 radius=0.04; visual mesh filename=meshes/R_thigh.STL
- link R_toe: geometry collision mesh filename=meshes/R_toe_old.STL; visual mesh filename=meshes/R_toe_old.STL
Joints:
- removed joint L_end_joint
- removed joint R_end_joint
- added joint Waist_joint: type fixed, parent Pelvis, child Torso, origin xyz=0 0 0.0825 rpy=0 0 0, axis 0 0 1, limit lower=-1.0472 upper=1.0472 effort=98 velocity=16
- joint L_calf_joint: limit lower=-1.571 upper=0.529 effort=105 velocity=50 -> lower=-1.571 upper=0.529 effort=98 velocity=15
- joint L_hip2_joint: limit lower=-0.26 upper=0.65 effort=125 velocity=50 -> lower=-0.18 upper=0.48 effort=98 velocity=23
- joint L_hip_joint: limit lower=-1.5 upper=1.5 effort=125 velocity=50 -> lower=-0.73 upper=0.73 effort=98 velocity=23; origin xyz=-0.0053471 0.1175 -0.0067 rpy=0 0 0 -> xyz=0 0.1175 -0.0067 rpy=0 0 0; parent base -> Pelvis
- joint L_thigh_joint: limit lower=-1.25 upper=1.1 effort=125 velocity=50 -> lower=-1.25 upper=1.1 effort=98 velocity=23; origin xyz=0.078 -0.014084 -0.0185 rpy=0 -0.78539816339 0 -> xyz=0.084 -0.0148 -0.0185 rpy=0 -0.78539816339 0
- joint L_toe_joint: limit lower=-0.3 upper=1.6 effort=30 velocity=50 -> lower=-0.3 upper=1.5 effort=25 velocity=11.5
- joint R_calf_joint: limit lower=-1.571 upper=0.529 effort=105 velocity=50 -> lower=-1.571 upper=0.529 effort=98 velocity=15
- joint R_hip2_joint: limit lower=-0.65 upper=0.26 effort=125 velocity=50 -> lower=-0.48 upper=0.18 effort=98 velocity=23
- joint R_hip_joint: limit lower=-1.5 upper=1.5 effort=125 velocity=50 -> lower=-0.73 upper=0.73 effort=98 velocity=23; origin xyz=-0.0053471 -0.1175 -0.0067 rpy=0 0 0 -> xyz=0 -0.1175 -0.0067 rpy=0 0 0; parent base -> Pelvis
- joint R_thigh_joint: limit lower=-1.25 upper=1.1 effort=125 velocity=50 -> lower=-1.25 upper=1.1 effort=98 velocity=23; origin xyz=0.078 0.014084 -0.0185 rpy=0 -0.78539816339 0 -> xyz=0.084 0.0148 -0.0185 rpy=0 -0.78539816339 0
- joint R_toe_joint: limit lower=-0.3 upper=1.6 effort=30 velocity=50 -> lower=-0.3 upper=1.5 effort=25 velocity=11.5
